File: 1200_MIC/1200_MIC/1200_MIC.sch (KiCad schematic (older format))
At the start: 122 parts, among them J1 +48V, J10 +MIC2-72, J11 GND-72, J12 -MIC2-72, J13 LINE2-73, J14 GND-73, J15 OUT1-74, J16 GND-70, J17 OUT2-75, J18 M/S-42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

Commit message: First version preamp 1200
Parts:
- removed C13, C41, C43, C45, C47, C51, C53, C7: C_0074, DVB_Capacitor_Film:C_2820, symbol DVB_C:C_0074
- removed C14, C4, C42, C44, C46, C48, C52, C54, C8: C_0072, DVB_Capacitors_Electrolytic:C_Radial_D12.5mm_H25.0mm_P5.00mm, symbol DVB_C:C_0072
- removed C25, C26: C_0076, DVB_Resistors:R_0402, symbol DVB_C:C_0076
- removed J1: +48V, DVB_Connectors:Solder_Pad_8x5, symbol Connector_Generic:Conn_01x01
- removed L1, L2, L3, L4, L5, L6: 10uH, symbol Device:L_Core_Iron
- removed R10, R7, R8, R9: R_0162, DVB_Resistors:R_0402, symbol DVB_R:R_0162
- removed R4, R6: R_0033, DVB_Resistors:R_0402, symbol DVB_R:R_0033
- added C13, C41, C43, C45, C47, C51, C53, C7: C_0075, DVB_Capacitors_Ceramic:C_0805, symbol DVB_C:C_0075
- added C14, C42, C44, C46, C48, C52, C54, C8: C_0078, DVB_Capacitors_Electrolytic:CP_Radial_D8.0mm_P3.50mm, symbol DVB_C:C_0078
- added C56: C_0002, DVB_Capacitors_Ceramic:C_0402, symbol DVB_C:C_0002
- added D1, D10, D11, D12, D2, D3, D4, D5, D6, D7, D8, D9: D_0022, DVB_Diodes:D_SOD-523, symbol DVB_D:D_0022
- added L1, L2, L3, L4, L5, L6: L_0001, Ferrite_THT:LairdTech_28C0236-0JW-10, symbol DVB_L:L_0001
- C10, C11, C16, C17: footprint DVB_Capacitors_Electrolytic:C_Radial_D12.5mm_H25.0mm_P5.00mm -> DVB_Capacitors_Electrolytic:CP_Radial_D12.5mm_P5.00mm
- J10, J11, J12, J13, J14, J15, J16, J17, J18, J2, J3, J4, J5, J6, J7, J8, J9: footprint DVB_Connectors:Solder_Pad_8x5 -> DVB_Connectors:stamped_contact_2.8mm
- Q1, Q3: Field1 N-chan -> FDN361BN
- Q2: Field1 P-chan -> FDN358P
- Q4: footprint DVB_SOT:SOT_23-6 -> DVB_SOT:SOT_23; Field1 P-chan -> MMBFJ176
- RV1, RV2: footprint Potentiometer_THT:Potentiometer_Omeg_PC16BU_Vertical -> DVB_Resistors:Potentiometer_Mono_Vertical
- RV3: value R_POT -> 10k; footprint Potentiometer_THT:Potentiometer_Omeg_PC16BU_Vertical -> DVB_Resistors:Potentiometer_Stereo_Vertical
Connections:
- net +4.9V: now also D1.1 (K), D11.1 (K), D3.1 (K), D5.1 (K), D7.1 (K), D9.1 (K)
- net -4.9V: now also D10.2 (A), D12.2 (A), D2.2 (A), D4.2 (A), D6.2 (A), D8.2 (A)
- net GND: now also RV3.3, RV3.6, C56.2; no longer RV3.3, RV3.6
- net LINE1: now also C7.1, C8.1
- net LINE2: now also C13.1, C14.1
- net MIC2+: now also C15.1, C16.1; no longer C17.1, C18.2
- net MIC2-: now also C17.1, C18.2; no longer C15.1, C16.1
- net MS: now also C56.1
- net OUT1: now also C51.2, C52.2
- net OUT2: now also C53.2, C54.2
- net at C11.2, C12.1: now also L3.1
- net at C10.2, C9.2: now also L2.1
- net at R5.1, U3.8 (Sns), U3.9 (VO): now also C43.1, C44.1
- net at R19.1, U3.12 (GS2): now also RV2.3; no longer RV1.3
- net at C20.1, R11.1, U3.4 (VIN-): now also D5.2 (A), D6.1 (K), L2.2
- net at C21.2, R13.1, U3.5 (VIN+): now also D1.2 (A), D2.1 (K), L3.2
- net at C19.1, R15.2, U1.5 (B+): now also D10.1 (K), D9.2 (A), L1.2
- net at R23.1, U1.7 (OUTB): now also C41.1, C42.1
- net at U5.1 (OUTA), U5.2 (A-): now also C51.1, C52.1
- net at R26.2, R28.2: now also RV3.4; no longer RV3.1
- net at R30.1: now also RV3.5; no longer RV3.2
- net at R27.2, R29.2: now also RV3.1; no longer RV3.4
- net at R31.1: now also RV3.2; no longer RV3.5
- net at U5.5 (B+), U5.7 (OUTB): now also C53.1, C54.1
- net at R26.1: now also C43.2, C44.2
- net at R28.1: now also C41.2, C42.2
- net at R19.2, R21.2: now also RV2.1, RV2.2; no longer RV1.1, RV1.2
- net at R20.2, R22.2: now also RV1.1, RV1.2; no longer RV2.1, RV2.2
- net at R25.1, U4.8 (Sns), U4.9 (VO): now also C47.1, C48.1
- net at C17.2, C18.1: now also L6.1
- net at C15.2, C16.2: now also L5.1
- net at R20.1, U4.12 (GS2): now also RV1.3; no longer RV2.3
- net at C23.1, R12.1: now also U4.5 (VIN+), D3.2 (A), D4.1 (K), L5.2; no longer U4.4 (VIN-)
- net at C24.2, R14.1: now also U4.4 (VIN-), D7.2 (A), D8.1 (K), L6.2; no longer U4.5 (VIN+)
- net at C22.1, R16.2, U2.5 (B+): now also D11.2 (A), D12.1 (K), L4.2
- net at R24.1, U2.7 (OUTB): now also C45.1, C46.1
- net at R27.1: now also C47.2, C48.2
- net at R29.1: now also C45.2, C46.2
- new net: C7.2, C8.2, L1.1
- new net: C13.2, C14.2, L4.1
Other:
- note added: "13.13.755 ETTINGER"
- moved on the sheet: C15, C16, C17, C18, C19, C20, C21, C22, C23, C24, J10, J11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
