File: 400_PW/400_PW.sch (KiCad schematic (older format))
At the start: 101 parts, among them J1 TESTBAT-14, J10 GNDBATT-4B, J11 GND-7_21_22_3B_28_51B_53_76, J2 ON/OFF-6A, J3 +7.5V-13_26_33_51A_54_104_6A, J4 +4.9V-10_36_80_83_93, J5 -4.9V, J6 +48V, J7 BATT-4A_6B, J8 15VIN-3A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

Commit message: Update schematics
Parts:
- added J12: TESTBAT-14, DVB_Connectors:Solder_Pad_8x5, symbol Connector_Generic:Conn_01x01
- added R21: R_0020, DVB_Resistors:R_0402, symbol DVB_R:R_0020
- J1, J10, J11, J2, J3, J4, J5, J6, J7, J8, J9: footprint (none) -> DVB_Connectors:Solder_Pad_8x5
- K1: footprint DVB_Connectors:Pol_Pin_Header_1x3-P2.54-RA -> Connector_JST:JST_EH_B3B-EH-A_1x03_P2.50mm_Vertical
- RV1: footprint (none) -> Potentiometer_THT:Potentiometer_Piher_PT-6-V_Vertical_Hole
Connections:
- net at U5.4 (*CHRG): now also R21.1
- new net CHG_LED: J12.1 (Pin_1), R21.2
- no-connect marks 5 -> 6
Other:
- moved on the sheet: J1, J10, J11, J2, J3, J4, J5, J6, J7, J8, J9, K1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

Commit message: Place components on 400_PW
Parts:
- removed J10: GNDBATT-4B, DVB_Connectors:Solder_Pad_8x5, symbol Connector_Generic:Conn_01x01
- removed J9: GNDAKKU-5, DVB_Connectors:Solder_Pad_8x5, symbol Connector_Generic:Conn_01x01
- added J13: GND, DVB_Connectors:Solder_Pad_8x5, symbol Connector_Generic:Conn_01x01
- J7: value BATT-4A_6B -> ON/OFF-4A_6B
Connections:
- net +BATT: no longer J7.1 (Pin_1)
- net GND: now also J13.1 (Pin_1)
- net VDD: now also J7.1 (Pin_1)
- no-connect marks 6 -> 4
Other:
- moved on the sheet: J11

Commit message: Update PW 400
Parts:
- removed K1: K_0008, Connector_JST:JST_EH_B3B-EH-A_1x03_P2.50mm_Vertical, symbol DVB_K:K_0008
- added C46: C_0002, DVB_Capacitors_Ceramic:C_0402, symbol DVB_C:C_0002
- added J9: ON/OFF-48V, DVB_Connectors:Solder_Pad_8x5, symbol Connector_Generic:Conn_01x01
- added K1: BATT, Connector_JST:JST_VH_B2P-VH_1x02_P3.96mm_Vertical, symbol Connector_Generic:Conn_01x02
- added R22: R_0034, DVB_Resistors:R_0402, symbol DVB_R:R_0034
- RV1: footprint Potentiometer_THT:Potentiometer_Piher_PT-6-V_Vertical_Hole -> Potentiometer_THT:Potentiometer_Piher_PT-10-V10_Vertical_Hole
Connections:
- net +7.5V: no longer U4.1 (~SDHN)
- net +BATT: now also K1.2 (Pin_2)
- net GND: now also C46.1, K1.1 (Pin_1), R22.2
- net NTC: no longer names the net of U5.8 (NTC)
- new net EN_48V: C46.2, J9.1 (Pin_1), R22.1, U4.1 (~SDHN)
- no-connect marks 4 -> 5
Changed lines of the file:
@@
 	4000 4075 4625 4075
-$Comp
-L DVB_K:K_0008 K1
-U 1 1 5DCB6BF7
-P 9325 3925
-F 0 "K1" H 9403 3966 50  0000 L CNN
-F 1 "K_0008" H 9325 3725 50  0001 C CNN
-F 2 "Connector_JST:JST_EH_B3B-EH-A_1x03_P2.50mm_Vertical" H 9325 3625 50  0001 C CNN
-F 3 "http://katalog.we-online.de/em/datasheet/6190xx11021.pdf" H 9325 3525 50  0001 C CNN
-F 4 "61900311021" H 9403 3875 50  0000 L CNN "Field4"
-F 5 "3p" H 9325 3425 50  0001 C CNN "Field5"
-F 6 "male" H 9325 3325 50  0001 C CNN "Field6"
-F 7 "RA" H 9325 3225 50  0001 C CNN "Field7"
-	1    9325 3925
-	1    0    0    1
-$EndComp
 $Comp
 L DVB_D:D_0026 D1
@@
 	0    1    -1   0
 $EndComp
-Text Label 7725 2475 2    39   ~ 0
-NTC
-Text Label 9125 3925 2    39   ~ 0
-NTC
 $Comp
 L DVB_Power:P_FLG #FLG0106
@@
 L DVB_Power:+BATT #PWR0131
 U 1 1 5DD93EC0
-P 9125 3825
-F 0 "#PWR0131" H 9125 3755 30  0001 C CNN
-F 1 "+BATT" H 9125 3963 30  0000 C CNN
-F 2 "" H 9125 3825 60  0001 C CNN
-F 3 "" H 9125 3825 60  0001 C CNN
-	1    9125 3825
+P 9125 3925
+F 0 "#PWR0131" H 9125 3855 30  0001 C CNN
+F 1 "+BATT" H 9125 4063 30  0000 C CNN
+F 2 "" H 9125 3925 60  0001 C CNN
+F 3 "" H 9125 3925 60  0001 C CNN
+	1    9125 3925
 	0    -1   1    0
 $EndComp
@@
 $EndComp
 $Comp
-L DVB_Power:+7.5V #PWR0167
-U 1 1 5E28746A
-P 2450 7100
-F 0 "#PWR0167" H 2450 7030 30  0001 C CNN
-F 1 "+7.5V" H 2450 7238 30  0000 C CNN
-F 2 "" H 2450 7100 60  0001 C CNN
-F 3 "" H 2450 7100 60  0001 C CNN
-	1    2450 7100
-	0    -1   -1   0
-$EndComp
-$Comp
 L DVB_Power:+7.5V #PWR0168
 U 1 1 5E288F03
@@
 F 0 "RV1" V 8560 4450 50  0000 C CNN
 F 1 "25K" V 8469 4450 50  0000 C CNN
-F 2 "Potentiometer_THT:Potentiometer_Piher_PT-6-V_Vertical_Hole" H 8675 4450 50  0001 C CNN
+F 2 "Potentiometer_THT:Potentiometer_Piher_PT-10-V10_Vertical_Hole" H 8675 4450 50  0001 C CNN
 F 3 "PT10LV10-253A2020-PM-S" H 8675 4450 50  0001 C CNN
 	1    8675 4450
@@
 	1    0    0    1
 $EndComp
-Connection ~ 9125 4025
 $Comp
 L DVB_Power:P_FLG #FLG0111
@@
 L DVB_Power:P_FLG #FLG0112
 U 1 1 5DBA782F
-P 9125 3825
-F 0 "#FLG0112" H 9125 3775 30  0001 C CNN
-F 1 "P_FLG" H 9125 3935 30  0000 C CNN
-F 2 "" H 9125 3825 50  0000 C CNN
-F 3 "" H 9125 3825 50  0000 C CNN
-	1    9125 3825
-	1    0    0    -1
-$EndComp
-Connection ~ 9125 3825
+P 9125 3925
+F 0 "#FLG0112" H 9125 3875 30  0001 C CNN
+F 1 "P_FLG" H 9125 4035 30  0000 C CNN
+F 2 "" H 9125 3925 50  0000 C CNN
+F 3 "" H 9125 3925 50  0000 C CNN
+	1    9125 3925
+	1    0    0    -1
+$EndComp
 $Comp
 L Connector_Generic:Conn_01x01 J12
@@
 	1    0    0    -1
 $EndComp
+$Comp
+L Connector_Generic:Conn_01x01 J9
+U 1 1 5DBC53A0
+P 9325 6200
+F 0 "J9" H 9405 6242 50  0000 L CNN
+F 1 "ON/OFF-48V" H 9405 6151 50  0000 L CNN
+F 2 "DVB_Connectors:Solder_Pad_8x5" H 9325 6200 50  0001 C CNN
+F 3 "~" H 9325 6200 50  0001 C CNN
+	1    9325 6200
+	1    0    0    -1
+$EndComp
+Text Label 9125 6200 2    50   ~ 0
+EN_48V
+Text Label 2225 7100 2    50   ~ 0
+EN_48V
+$Comp
+L DVB_C:C_0002 C46
+U 1 1 5DBC86F4
+P 2225 7250
+F 0 "C46" H 2325 7325 50  0000 L CNN
+F 1 "C_0002" H 2225 6950 50  0001 C CNN
+F 2 "DVB_Capacitors_Ceramic:C_0402" H 2225 6800 50  0001 C CNN
+F 3 "generic" H 2225 6875 50  0001 C CNN
+F 4 "100nF" H 2325 7250 50  0000 L CNN "Field1"
+F 5 "C-0402" H 2325 7100 50  0001 L CNN "Field2"
+F 6 "25V" H 2325 7175 50  0000 L CNN "Field3"
+F 7 "X7R" H 2325 7025 50  0001 L CNN "Field4"
+	1    2225 7250
+	-1   0    0    1
+$EndComp
+$Comp
+L DVB_Power:GND #PWR03
+U 1 1 5DBC92ED
+P 2450 7400
+F 0 "#PWR03" H 2450 7240 30  0001 C CNN
+F 1 "GND" H 2450 7290 30  0000 C CNN
+F 2 "" H 2350 7050 50  0001 C CNN
+F 3 "" H 2450 7150 50  0001 C CNN
+	1    2450 7400
+	1    0    0    -1
+$EndComp
+$Comp
+L DVB_Power:GND #PWR02
+U 1 1 5DBC95DA
+P 2225 7400
+F 0 "#PWR02" H 2225 7240 30  0001 C CNN
+F 1 "GND" H 2225 7290 30  0000 C CNN
+F 2 "" H 2125 7050 50  0001 C CNN
+F 3 "" H 2225 7150 50  0001 C CNN
+	1    2225 7400
+	1    0    0    -1
+$EndComp
+Wire Wire Line
+	2225 7100 2450 7100
+$Comp
+L DVB_R:R_0034 R22
+U 1 1 5DBD3D2B
+P 2450 7250
+F 0 "R22" H 2525 7200 50  0000 L CNN
+F 1 "R_0034" H 2450 7050 50  0001 C CNN
+F 2 "DVB_Resistors:R_0402" H 2450 6900 50  0001 C CNN
+F 3 "generic" H 2450 6975 50  0001 C CNN
+F 4 "100k" V 2450 7150 50  0000 L CNN "Field4"
+F 5 "1%" V 2200 7150 50  0001 L CNN "Field5"
+F 6 "100mW" V 2275 7150 50  0001 L CNN "Field6"
+	1    2450 7250
+	1    0    0    -1
+$EndComp
+Connection ~ 2450 7100
+$Comp
+L Connector_Generic:Conn_01x02 K1
+U 1 1 5DE4300F
+P 9325 4025
+F 0 "K1" H 9450 3925 50  0000 C CNN
+F 1 "BATT" H 9625 4025 50  0000 C CNN
+F 2 "Connector_JST:JST_VH_B2P-VH_1x02_P3.96mm_Vertical" H 9325 4025 50  0001 C CNN
+F 3 "~" H 9325 4025 50  0001 C CNN
+	1    9325 4025
+	1    0    0    1
+$EndComp
+Connection ~ 9125 3925
+Connection ~ 9125 4025
+NoConn ~ 7725 2475
 $EndSCHEMATC

Commit message: 600 MIC v1.0.0
Other:
- note added: "ERREUR!"
Changed lines of the file:
@@
 EESchema Schematic File Version 4
-LIBS:400_PW-cache
 EELAYER 30 0
 EELAYER END
@@
 Connection ~ 9125 4025
 NoConn ~ 7725 2475
+Text Notes 10900 1375 0    50   ~ 0
+ERREUR!
 $EndSCHEMATC
